File: pcb/vl6180x.brd (EAGLE design)
At the start: 8.3 x 15.9 mm, 5 parts, among them J1 6PINBOARDEDGE, U1 STPROXSENSOR

Commit message: Fixed 2.8v regulator pinout
Parts:
- C1: value 0.1nF -> 0.1uF
- C2: value 4.7nF -> 4.7uF
Changed lines of the file:
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@@
 </autorouter>
 <elements>
-<element name="C1" library="SparkFun-Passives" package="0603-CAP" value="0.1nF" x="6.6675" y="12.7" rot="MR270"/>
-<element name="C2" library="SparkFun-Passives" package="0603-CAP" value="4.7nF" x="4.1275" y="12.7" rot="MR270"/>
+<element name="C1" library="SparkFun-Passives" package="0603-CAP" value="0.1uF" x="6.6675" y="12.7" rot="MR270"/>
+<element name="C2" library="SparkFun-Passives" package="0603-CAP" value="4.7uF" x="4.1275" y="12.7" rot="MR270"/>
 <element name="R1" library="SparkFun-Passives" package="0603-RES" value="47k" x="1.5875" y="12.7" rot="MR270"/>
 <element name="U1" library="Nick'sEagle" package="STPROXSENSOR" value="STPROXSENSOR" x="4.1275" y="12.7" smashed="yes"/>
