File: pcb/lipo-shutoff.brd (EAGLE design)
At the start: 21 x 7.6 mm, 10 parts, among them Q1 AON6411, SW1 FSM4JSMA, U1 LT6703-2

Commit message: Fixed lipo cutoff board
Connections:
- net N$1: now also Q1.1, Q1.2, Q1.3; no longer Q1.5, Q1.6, Q1.7, Q1.8, Q1.PAD
- net N$4: now also Q1.5, Q1.6, Q1.7, Q1.8, Q1.PAD; no longer Q1.1, Q1.2, Q1.3
Changed lines of the file:
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@@
 <signal name="N$1">
 <contactref element="JP1" pad="1"/>
-<contactref element="Q1" pad="5"/>
-<contactref element="Q1" pad="6"/>
-<contactref element="Q1" pad="7"/>
-<contactref element="Q1" pad="8"/>
-<contactref element="Q1" pad="PAD"/>
 <contactref element="R3" pad="2"/>
 <polygon width="0.254" layer="16" thermals="no">
@@
 <vertex x="8.255" y="7.62"/>
 </polygon>
-</signal>
-<signal name="N$4">
 <contactref element="Q1" pad="1"/>
 <contactref element="Q1" pad="2"/>
 <contactref element="Q1" pad="3"/>
+<wire x1="9.735" y1="3.81" x2="9.735" y2="5.08" width="0" layer="19" extent="16-16"/>
+<wire x1="9.735" y1="2.54" x2="9.735" y2="3.81" width="0" layer="19" extent="16-16"/>
+<wire x1="4.865" y1="6.35" x2="9.735" y2="5.08" width="0" layer="19" extent="16-16"/>
+<wire x1="1.905" y1="5.207" x2="4.865" y2="6.35" width="0" layer="19" extent="16-16"/>
+</signal>
+<signal name="N$4">
 <contactref element="JP2" pad="1"/>
 <contactref element="U1" pad="2"/>
@@
 <vertex x="8.89" y="7.62"/>
 </polygon>
+<contactref element="Q1" pad="5"/>
+<contactref element="Q1" pad="PAD"/>
+<contactref element="Q1" pad="8"/>
+<contactref element="Q1" pad="7"/>
+<contactref element="Q1" pad="6"/>
+<wire x1="15.875" y1="2.96" x2="19.05" y2="5.207" width="0" layer="19" extent="16-16"/>
+<wire x1="6.525" y1="3.175" x2="11.005" y2="1.27" width="0" layer="19" extent="16-16"/>
+<wire x1="4.235" y1="3.81" x2="6.525" y2="3.175" width="0" layer="19" extent="16-16"/>
+<wire x1="4.235" y1="5.08" x2="4.235" y2="3.81" width="0" layer="19" extent="16-16"/>
+<wire x1="4.235" y1="2.54" x2="4.235" y2="3.81" width="0" layer="19" extent="16-16"/>
+<wire x1="4.235" y1="1.27" x2="4.235" y2="2.54" width="0" layer="19" extent="16-16"/>
 </signal>
 <signal name="N$3">
